File: TEENSY_4.0_AUDIO_TOOLKIT.sch (KiCad schematic (older format))
At the start: 43 parts, among them U3 Teensy4.0, U4C1 22 uF, U4C2 0.47uF, U4C3 0.47uF, U4C4 22 uF

Commit message: Update
Parts:
- added R14: 220R, Resistor_SMD:R_0603_1608Metric_Pad1.05x0.95mm_HandSolder, symbol Device:R_Small
Connections:
- net OUT1B: now also R14.1
Changed lines of the file:
@@
 Wire Wire Line
 	8000 7050 8200 7050
+Text GLabel 4550 3400 2    50   Input ~ 0
+OUT1B
+$Comp
+L Device:R_Small R14
+U 1 1 5E97C255
+P 4450 3400
+F 0 "R14" V 4395 3295 20  0000 L CNN
+F 1 "220R" V 4464 3335 20  0000 L CNN
+F 2 "Resistor_SMD:R_0603_1608Metric_Pad1.05x0.95mm_HandSolder" H 4450 3400 50  0001 C CNN
+F 3 "~" H 4450 3400 50  0001 C CNN
+F 4 "SM0603_Resistor" V 4500 3405 20  0001 C CNN "Package / Case"
+	1    4450 3400
+	0    1    1    0
+$EndComp
 $EndSCHEMATC

Commit message: update
Parts:
- removed R14: 220R, Resistor_SMD:R_0603_1608Metric_Pad1.05x0.95mm_HandSolder, symbol Device:R_Small
- added J?: Conn_02x05_Odd_Even, symbol Connector_Generic:Conn_02x05_Odd_Even
- added J?: Conn_01x03_MountingPin, symbol Connector_Generic_MountingPin:Conn_01x03_MountingPin
- added JP_MOSI1, JP_SCK1: SolderJumper_3_Bridged12, symbol Jumper:SolderJumper_3_Bridged12
Connections:
- net 5V: now also J?.2 (Pin_2)
- net GND: now also J?.1 (Pin_1), J?.4 (Pin_4)
- net VIN: now also J?.2 (Pin_2)
- net SPI_CS: now reaches U3.12 (10_CS_MQSR)
- net SPI_CS: now also J?.7 (Pin_7)
- net SPI_MOSI: now reaches U3.13 (11_MOSI_CTX1)
- net SPI_MOSI: now also J?.5 (Pin_5)
- net SPI_MISO: now reaches U3.14 (12_MISO_MQSL)
- net SPI_MISO: now also J?.3 (Pin_3)
- net SPI_SCK: now reaches U3.20 (13_SCK_CRX1_LED)
- net SPI_SCK: now also J?.9 (Pin_9), JP_MOSI1.2 (C), JP_SCK1.2 (C)
- new net ?: J?.3 (Pin_3)
- new net INT: J?.8 (Pin_8)
- new net MOSI3: JP_MOSI1.3 (B)
- new net MOSI4: JP_MOSI1.1 (A)
- new net RST: J?.6 (Pin_6)
- new net SCK3: JP_SCK1.1 (A)
- new net SCK4: JP_SCK1.3 (B)
Other:
- note added: "EXPRESSION PEDALS"
- note added: "FAN HEADER"
- note added: "SPI"
- note added: "https://allpinouts.org/pinouts/connectors/motherboards/motherboard-cpu-3-pin-fan-connector/"
Changed lines of the file:
@@
 Wire Wire Line
 	8000 7050 8200 7050
-Text GLabel 4550 3400 2    50   Input ~ 0
-OUT1B
 $Comp
-L Device:R_Small R14
-U 1 1 5E97C255
-P 4450 3400
-F 0 "R14" V 4395 3295 20  0000 L CNN
-F 1 "220R" V 4464 3335 20  0000 L CNN
-F 2 "Resistor_SMD:R_0603_1608Metric_Pad1.05x0.95mm_HandSolder" H 4450 3400 50  0001 C CNN
-F 3 "~" H 4450 3400 50  0001 C CNN
-F 4 "SM0603_Resistor" V 4500 3405 20  0001 C CNN "Package / Case"
-	1    4450 3400
-	0    1    1    0
+L Connector_Generic:Conn_02x05_Odd_Even J?
+U 1 1 5E9B251E
+P 13950 3900
+F 0 "J?" H 14000 4317 50  0000 C CNN
+F 1 "Conn_02x05_Odd_Even" H 14000 4226 50  0000 C CNN
+F 2 "" H 13950 3900 50  0001 C CNN
+F 3 "~" H 13950 3900 50  0001 C CNN
+	1    13950 3900
+	1    0    0    -1
 $EndComp
+Text GLabel 14250 3700 2    50   Input ~ 0
+VIN
+Text GLabel 14250 3900 2    50   Input ~ 0
+RST
+Text GLabel 14250 3800 2    50   Input ~ 0
+GND
+Text GLabel 14250 4000 2    50   Input ~ 0
+INT
+Text GLabel 13750 4100 0    50   Input ~ 0
+SPI_SCK
+Text GLabel 13750 3900 0    50   Input ~ 0
+SPI_MOSI
+Text GLabel 13750 4000 0    50   Input ~ 0
+SPI_CS
+Text GLabel 13750 3800 0    50   Input ~ 0
+SPI_MISO
+Text Notes 13905 3074 0    79   ~ 16
+SPI
+$Comp
+L Jumper:SolderJumper_3_Bridged12 JP_MOSI1
+U 1 1 5E9F4B01
+P 9800 3550
+F 0 "JP_MOSI1" H 9800 3663 50  0000 C CNN
+F 1 "SolderJumper_3_Bridged12" H 9800 3664 50  0001 C CNN
+F 2 "" H 9800 3550 50  0001 C CNN
+F 3 "~" H 9800 3550 50  0001 C CNN
+	1    9800 3550
+	1    0    0    -1
+$EndComp
+$Comp
+L Jumper:SolderJumper_3_Bridged12 JP_SCK1
+U 1 1 5E9F5F41
+P 9850 4050
+F 0 "JP_SCK1" H 9850 4163 50  0000 C CNN
+F 1 "SolderJumper_3_Bridged12" H 9850 4164 50  0001 C CNN
+F 2 "" H 9850 4050 50  0001 C CNN
+F 3 "~" H 9850 4050 50  0001 C CNN
+	1    9850 4050
+	1    0    0    -1
+$EndComp
+Text GLabel 9650 4050 0    50   Input ~ 0
+SCK3
+Text GLabel 10050 4050 2    50   Input ~ 0
+SCK4
+Text GLabel 10000 3550 2    50   Input ~ 0
+MOSI3
+Text GLabel 9600 3550 0    50   Input ~ 0
+MOSI4
+Text GLabel 9850 4200 2    50   Input ~ 0
+SPI_SCK
+Text GLabel 9800 3700 2    50   Input ~ 0
+SPI_SCK
+Text GLabel 1650 3300 0    50   Input ~ 0
+SPI_MOSI
+Text GLabel 1650 3400 0    50   Input ~ 0
+SPI_MISO
+Text GLabel 1650 3200 0    50   Input ~ 0
+SPI_CS
+Text GLabel 1650 4000 0    50   Input ~ 0
+SPI_SCK
+Text Notes 12605 674  0    79   ~ 16
+EXPRESSION PEDALS
+Text Notes 13705 4524 0    79   ~ 16
+FAN HEADER
+$Comp
+L Connector_Generic_MountingPin:Conn_01x03_MountingPin J?
+U 1 1 5EA94C28
+P 14150 4950
+F 0 "J?" H 14238 4914 50  0000 L CNN
+F 1 "Conn_01x03_MountingPin" H 14100 3950 50  0000 L CNN
+F 2 "" H 14150 4950 50  0001 C CNN
+F 3 "~" H 14150 4950 50  0001 C CNN
+	1    14150 4950
+	1    0    0    -1
+$EndComp
+Text GLabel 13950 4850 0    50   Input ~ 0
+GND
+Text GLabel 13950 4950 0    50   Input ~ 0
+5V
+Text GLabel 13950 5050 0    50   Input ~ 0
+?
+Text Notes 8550 4950 0    39   ~ 0
+https://allpinouts.org/pinouts/connectors/motherboards/motherboard-cpu-3-pin-fan-connector/
 $EndSCHEMATC
